Commit message: Fix code

File: urdf/robot.urdf (robot description, URDF)
Before this commit: robot warehouse_robot, 8 links, 7 joints
Links:
- removed link caster_wheel_link
- removed link wheel_left_link
- removed link wheel_right_link
- added link base_footprint
- added link caster_wheel, mass 0.5; collision sphere radius=0.05; visual sphere radius=0.05
- added link caster_wheel_front, mass 0.5; collision sphere radius=0.05; visual sphere radius=0.05
- added link laser_frame, mass 0.2; collision cylinder length=0.05 radius=0.05; visual cylinder length=0.05 radius=0.05
- added link left_wheel, mass 1.0; collision cylinder length=0.05 radius=0.1; visual cylinder length=0.05 radius=0.1
- added link right_wheel, mass 1.0; collision cylinder length=0.05 radius=0.1; visual cylinder length=0.05 radius=0.1
- link arm_base_link: geometry collision cylinder length=0.02 radius=0.04; visual cylinder length=0.02 radius=0.04
- link arm_link1: mass 0.4 -> 0.5; geometry collision box size=0.04 0.04 0.3; visual box size=0.04 0.04 0.3
- link arm_link2: mass 0.3 -> 0.4; geometry collision box size=0.03 0.03 0.3; visual box size=0.03 0.03 0.3
- link base_link: mass 5.0 -> 10.0; geometry collision box size=0.5 0.3 0.2; visual box size=0.5 0.3 0.2
- link gripper_touchpoint: geometry 
Joints:
- removed joint arm_elbow_joint
- removed joint arm_shoulder_joint
- removed joint wheel_left_joint
- removed joint wheel_right_joint
- added joint base_footprint_joint: type fixed, parent base_footprint, child base_link, origin xyz=0 0 0.2 rpy=0 0 0
- added joint caster_wheel_front_joint: type fixed, parent base_link, child caster_wheel_front, origin xyz=0.2 0 -0.15 rpy=0 0 0
- added joint joint1: type revolute, parent arm_base_link, child arm_link1, origin xyz=0 0 0.01 rpy=0 0 0, axis 0 1 0, limit lower=-1.57 upper=1.57 effort=10 velocity=1.0
- added joint joint2: type revolute, parent arm_link1, child arm_link2, origin xyz=0 0 0.3 rpy=0 0 0, axis 0 1 0, limit lower=-1.57 upper=1.57 effort=10 velocity=1.0
- added joint laser_joint: type fixed, parent base_link, child laser_frame, origin xyz=0.15 0 0.15 rpy=0 0 0
- added joint left_wheel_joint: type continuous, parent base_link, child left_wheel, origin xyz=0 0.175 -0.1 rpy=-1.5708 0 0, axis 0 0 1
- added joint right_wheel_joint: type continuous, parent base_link, child right_wheel, origin xyz=0 -0.175 -0.1 rpy=-1.5708 0 0, axis 0 0 1
- joint arm_base_joint: origin xyz=0 0 0.10 rpy=0 0 0 -> xyz=0 0 0.1 rpy=0 0 0
- joint caster_wheel_joint: child caster_wheel_link -> caster_wheel; origin xyz=-0.20 0 -0.06 rpy=0 0 0 -> xyz=-0.2 0 -0.15 rpy=0 0 0
- joint gripper_touchpoint_joint: origin xyz=0 0 0.20 rpy=0 0 0 -> xyz=0 0 0.3 rpy=0 0 0
